Commit message: fixed rear lidar orientation to z=1.54

File: urdf/amr.urdf.xacro (robot description, xacro)
@@ -94,5 +94,5 @@
         <parent link="main_body_link"/>
         <child link="lidar_rear_link"/>
-        <origin xyz="-0.377 0.0 0.0" rpy="0.0 0.0 0.0"/>
+        <origin xyz="-0.377 0.0 0.0" rpy="0.0 0.0 1.54"/>
     </joint>
     <link name="ceiling_main_body_link">
